File: examples/sample.kicad_sch (KiCad schematic)
At the start: 4 parts, among them Q1 2N3904

Commit message: Fix parser
Exclude lib_symbols templates from placed components, recover pin geometry
from library definitions, and rebuild net connectivity with union-find over
wire segments so T-junctions and no-connect markers resolve correctly.

Co-Authored-By: Devin AI <158243242+devin-ai-integration[bot]@users.noreply.github.com>
Connections:
- net GND: now also C1.2
- new net VIN: R1.1
- new net VOUT: C1.1, R1.2, R2.1
- no-connect marks 0 -> 1
Changed lines of the file:
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@@
 	(wire
 		(pts
-			(xy 100 80) (xy 120 80)
+			(xy 110 80) (xy 116.19 80)
 		)
 		(stroke
@@
 	(wire
 		(pts
-			(xy 120 80) (xy 120 100)
+			(xy 123.81 80) (xy 140 80)
 		)
 		(stroke
@@
 	(wire
 		(pts
-			(xy 120 100) (xy 140 100)
+			(xy 140 80) (xy 140 86.19)
 		)
 		(stroke
@@
 	(wire
 		(pts
-			(xy 140 100) (xy 160 100)
+			(xy 140 80) (xy 156.19 80)
 		)
 		(stroke
@@
 	(wire
 		(pts
-			(xy 160 100) (xy 160 120)
+			(xy 140 93.81) (xy 140 100)
 		)
 		(stroke
@@
 		(uuid "w005")
 	)
-	(wire
-		(pts
-			(xy 100 80) (xy 100 60)
-		)
-		(stroke
-			(width 0)
-			(type default)
-		)
-		(uuid "w006")
-	)
-	(wire
-		(pts
-			(xy 160 120) (xy 160 140)
-		)
-		(stroke
-			(width 0)
-			(type default)
-		)
-		(uuid "w007")
+	(junction
+		(at 140 80)
+		(diameter 0)
+		(uuid "j001")
 	)
 	(label "VIN"
-		(at 100 60 0)
+		(at 110 80 0)
 		(effects
 			(font
@@
 	)
 	(label "VOUT"
-		(at 160 120 0)
+		(at 140 80 0)
 		(effects
 			(font
@@
 		(uuid "lbl002")
 	)
-	(global_label "GND"
-		(at 160 140 0)
-		(shape input)
-		(effects
-			(font
-				(size 1.27 1.27)
-			)
-			(justify left bottom)
-		)
-		(uuid "glbl001")
+	(no_connect
+		(at 210 100)
+		(uuid "nc001")
+	)
+	(symbol
+		(lib_id "power:GND")
+		(at 140 100 0)
+		(unit 1)
+		(in_bom yes)
+		(on_board yes)
+		(dnp no)
+		(uuid "sym005")
+		(property "Reference" "#PWR01"
+			(at 140 106 0)
+			(effects
+				(font
+					(size 1.27 1.27)
+				)
+				(hide yes)
+			)
+		)
+		(property "Value" "GND"
+			(at 140 105 0)
+			(effects
+				(font
+					(size 1.27 1.27)
+				)
+			)
+		)
+		(pin "1"
+			(uuid "pin010")
+		)
 	)
 	(symbol
 		(lib_id "Device:R")
-		(at 120 80 0)
+		(at 120 80 90)
 		(unit 1)
 		(exclude_from_sim no)
@@
 		(uuid "sym001")
 		(property "Reference" "R1"
-			(at 122 77 0)
+			(at 120 76 0)
 			(effects
 				(font
@@
 		)
 		(property "Value" "10k"
-			(at 122 83 0)
+			(at 120 84 0)
 			(effects
 				(font
@@
 		(pin "1"
 			(uuid "pin001")
-			(at 100 80 0)
-			(effects
-				(font
-					(size 1.27 1.27)
-				)
-			)
 		)
 		(pin "2"
 			(uuid "pin002")
-			(at 140 80 0)
-			(effects
-				(font
-					(size 1.27 1.27)
-				)
-			)
 		)
 	)
 	(symbol
 		(lib_id "Device:C")
-		(at 160 100 0)
+		(at 140 90 0)
 		(unit 1)
 		(exclude_from_sim no)
@@
 		(uuid "sym002")
 		(property "Reference" "C1"
-			(at 162 97 0)
+			(at 143 88 0)
 			(effects
 				(font
@@
 		)
 		(property "Value" "100n"
-			(at 162 103 0)
+			(at 143 92 0)
 			(effects
 				(font
@@
 		)
 		(property "Footprint" "Capacitor_SMD:C_0805_2012Metric"
-			(at 160 100 0)
+			(at 140 90 0)
 			(effects
 				(font
@@
 		)
 		(property "Sim.Device" "C"
-			(at 160 100 0)
+			(at 140 90 0)
 			(effects
 				(font
@@
 		)
 		(property "Sim.Pins" "1=passive 2=passive"
-			(at 160 100 0)
+			(at 140 90 0)
 			(effects
 				(font
@@
 		(pin "1"
 			(uuid "pin003")
-			(at 140 100 0)
-			(effects
-				(font
-					(size 1.27 1.27)
-				)
-			)
 		)
 		(pin "2"
 			(uuid "pin004")
-			(at 160 120 0)
-			(effects
-				(font
-					(size 1.27 1.27)
-				)
-			)
 		)
 	)
 	(symbol
 		(lib_id "Device:R")
-		(at 120 100 0)
+		(at 160 80 90)
 		(unit 1)
 		(exclude_from_sim no)
@@
 		(uuid "sym003")
 		(property "Reference" "R2"
-			(at 122 97 0)
+			(at 160 76 0)
 			(effects
 				(font
@@
 		)
 		(property "Value" "~"
-			(at 122 103 0)
+			(at 160 84 0)
 			(effects
 				(font
@@
 		)
 		(property "Footprint" ""
-			(at 120 100 0)
+			(at 160 80 0)
 			(effects
 				(font
@@
 		(pin "1"
 			(uuid "pin005")
-			(at 120 100 0)
-			(effects
-				(font
-					(size 1.27 1.27)
-				)
-			)
 		)
 		(pin "2"
 			(uuid "pin006")
-			(at 120 100 0)
-			(effects
-				(font
-					(size 1.27 1.27)
-				)
-			)
 		)
 	)
@@
 			(uuid "pin007")
 			(at 190 100 0)
-			(effects
-				(font
-					(size 1.27 1.27)
-				)
-			)
 		)
 		(pin "2"
 			(uuid "pin008")
 			(at 200 110 0)
-			(effects
-				(font
-					(size 1.27 1.27)
-				)
-			)
 		)
 		(pin "3"
 			(uuid "pin009")
 			(at 210 100 0)
-			(effects
-				(font
-					(size 1.27 1.27)
-				)
-			)
-		)
-	)
+		)
+	)
